File: kicad/GlyphMatrix_Top.kicad_pcb (KiCad board)
At the start: 2 copper layers, 298.3 x 128.6 mm, 74 parts

Commit message: Silk Screen
Other:
- outline, holes or cut-outs redrawn
- board text added: "Caps Lock"
- board text added: "OminCode:9001 - GlyphMatrix"
- board text added: "Power"
