File: kicad/GlyphMatrix_Plate.kicad_pcb (KiCad board)
At the start: 2 copper layers, 298.3 x 128.6 mm, 6 parts

Commit message: Silk Screen
Other:
- outline, holes or cut-outs redrawn
- board text added: "RESET"
- board text added: "UPDATE"

Commit message: Silk screen for plates
Other:
- board text added: "OminCode:9001 202507.13"
- board text added: "OmniCode:9001-GlyphMatrix"
- board text removed: "OminCode:9001 202507.12"
