File: kicad/GlyphMatrix-keymatrix.kicad_sch (KiCad schematic)
At the start: 169 parts

Commit message: artwork #2
Connections:
- net COL0: now also S13.2, S66.2, S69.2, S70.2, S71.2, S73.2; no longer S21.2, S33.2, S45.2, S56.2, S7.2
- net COL1: now also S12.2, S26.2, S38.2; no longer S22.2, S34.2, S46.2, S57.2, S8.2
- net COL2: now also S11.2, S25.2, S37.2, S49.2, S63.2; no longer S23.2, S35.2, S47.2, S58.2, S61.2, S9.2
- net COL3: now also S48.2; no longer S48.1
- net COL4: now also POGO3.7 (Pin_7), POGO4.1 (Pin_1), S23.2, S35.2, S47.2, S58.2, S61.2, S9.2; no longer POGO3.5 (Pin_5), POGO4.3 (Pin_3), S11.2, S25.2, S37.2, S49.2, S63.2
- net COL5: now also S22.2, S34.2, S46.2, S57.2, S8.2; no longer S12.2, S26.2, S38.2
- net COL6: now also POGO3.5 (Pin_5), POGO4.3 (Pin_3), S21.2, S33.2, S45.2, S56.2, S7.2; no longer POGO3.7 (Pin_7), POGO4.1 (Pin_1), S13.2, S66.2, S69.2, S70.2, S71.2, S73.2
- net at D48.2 (A): now also S48.1; no longer S48.2
Other:
- moved on the sheet: S48
Changed lines of the file:
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@@
 	)
 	(junction
+		(at 246.38 138.43)
+		(diameter 0)
+		(color 0 0 0 0)
+	)
+	(junction
 		(at 246.38 116.586)
 		(diameter 0)
@@
 	)
 	(junction
-		(at 246.38 138.43)
-		(diameter 0)
-		(color 0 0 0 0)
-	)
-	(junction
 		(at 251.46 151.13)
 		(diameter 0)
@@
 	(wire
 		(pts
+			(xy 246.38 116.586) (xy 246.38 138.43)
+		)
+		(stroke
+			(width 0)
+			(type default)
+		)
+	)
+	(wire
+		(pts
 			(xy 234.95 107.188) (xy 251.46 107.188)
 		)
@@
 	(wire
 		(pts
-			(xy 246.38 116.586) (xy 246.38 138.43)
-		)
-		(stroke
-			(width 0)
-			(type default)
-		)
-	)
-	(wire
-		(pts
 			(xy 90.424 193.802) (xy 106.934 193.802)
 		)
@@
 	(wire
 		(pts
-			(xy 246.38 138.43) (xy 246.38 159.766)
-		)
-		(stroke
-			(width 0)
-			(type default)
-		)
-	)
-	(wire
-		(pts
 			(xy 101.854 94.488) (xy 101.854 116.586)
 		)
@@
 	(wire
 		(pts
+			(xy 246.38 138.43) (xy 246.38 159.766)
+		)
+		(stroke
+			(width 0)
+			(type default)
+		)
+	)
+	(wire
+		(pts
 			(xy 165.608 94.488) (xy 165.608 116.586)
 		)
@@
 		)
 	)
-	(global_label "COL4"
+	(global_label "COL6"
 		(shape input)
 		(at 379.73 128.524 0)
@@
 		)
 	)
-	(global_label "COL5"
+	(global_label "COL1"
 		(shape input)
 		(at 278.384 58.674 90)
@@
 		)
 	)
-	(global_label "COL6"
+	(global_label "COL0"
 		(shape input)
 		(at 293.624 58.674 90)
@@
 		)
 	)
-	(global_label "COL4"
+	(global_label "COL6"
 		(shape input)
 		(at 33.782 128.524 180)
@@
 		)
 	)
-	(global_label "COL6"
+	(global_label "COL4"
 		(shape input)
 		(at 379.73 133.604 0)
@@
 		)
 	)
-	(global_label "COL1"
+	(global_label "COL5"
 		(shape input)
 		(at 214.63 58.674 90)
@@
 		)
 	)
-	(global_label "COL4"
+	(global_label "COL2"
 		(shape input)
 		(at 261.874 58.674 90)
@@
 		)
 	)
-	(global_label "COL6"
+	(global_label "COL4"
 		(shape input)
 		(at 33.782 133.604 180)
@@
 		)
 	)
-	(global_label "COL2"
+	(global_label "COL4"
 		(shape input)
 		(at 229.87 58.674 90)
@@
 		)
 	)
-	(global_label "COL0"
+	(global_label "COL6"
 		(shape input)
 		(at 198.12 58.674 90)
@@
 	(symbol
 		(lib_id "TB2086_KEYSWITCH:SW_MX_HS")
-		(at 248.92 140.97 0)
+		(at 248.92 140.97 270)
+		(mirror x)
 		(unit 1)
 		(exclude_from_sim no)
@@
 		(dnp no)
 		(property "Reference" "S48"
-			(at 248.92 134.112 0)
+			(at 255.778 140.97 0)
 			(effects
 				(font
@@
 		)
 		(property "Value" "SW_MX_HS"
-			(at 248.92 136.652 0)
+			(at 253.238 140.97 0)
 			(effects
 				(font
@@
 		)
 		(property "LCSC" "C9900021274"
-			(at 248.92 134.112 0)
+			(at 255.778 140.97 0)
 			(effects
 				(font

Commit message: changed screw sizes
Parts:
- H1, H2, H3, H4, H5, H6, H7, H8: footprint TB2086_MISC:MountingHole_3.2mm_Pad -> TB2086_MISC:MountingHole_2.2mm_M2_Pad
Changed lines of the file:
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@@
 			)
 		)
-		(property "Footprint" "TB2086_MISC:MountingHole_3.2mm_Pad"
+		(property "Footprint" "TB2086_MISC:MountingHole_2.2mm_M2_Pad"
 			(at 83.566 249.174 0)
 			(effects
@@
 			)
 		)
-		(property "Footprint" "TB2086_MISC:MountingHole_3.2mm_Pad"
+		(property "Footprint" "TB2086_MISC:MountingHole_2.2mm_M2_Pad"
 			(at 83.566 260.35 0)
 			(effects
@@
 			)
 		)
-		(property "Footprint" "TB2086_MISC:MountingHole_3.2mm_Pad"
+		(property "Footprint" "TB2086_MISC:MountingHole_2.2mm_M2_Pad"
 			(at 83.566 231.648 0)
 			(effects
@@
 			)
 		)
-		(property "Footprint" "TB2086_MISC:MountingHole_3.2mm_Pad"
+		(property "Footprint" "TB2086_MISC:MountingHole_2.2mm_M2_Pad"
 			(at 83.566 237.744 0)
 			(effects
@@
 			)
 		)
-		(property "Footprint" "TB2086_MISC:MountingHole_3.2mm_Pad"
+		(property "Footprint" "TB2086_MISC:MountingHole_2.2mm_M2_Pad"
 			(at 83.566 218.948 0)
 			(effects
@@
 			)
 		)
-		(property "Footprint" "TB2086_MISC:MountingHole_3.2mm_Pad"
+		(property "Footprint" "TB2086_MISC:MountingHole_2.2mm_M2_Pad"
 			(at 83.566 243.078 0)
 			(effects
@@
 			)
 		)
-		(property "Footprint" "TB2086_MISC:MountingHole_3.2mm_Pad"
+		(property "Footprint" "TB2086_MISC:MountingHole_2.2mm_M2_Pad"
 			(at 83.566 225.044 0)
 			(effects
@@
 			)
 		)
-		(property "Footprint" "TB2086_MISC:MountingHole_3.2mm_Pad"
+		(property "Footprint" "TB2086_MISC:MountingHole_2.2mm_M2_Pad"
 			(at 83.566 254.254 0)
 			(effects

Commit message: kibot
Parts:
- LED2: LCSC C84264 -> C965805
- S1, S10, S11, S12, S13, S14, S15, S16, S17, S18, S19, S2, S20, S21, S22, S23, S24, S25, S26, S27, S28, S29, S3, S30, S31, S32, S33, S34, S35, S36, S37, S38, S39, S4, S40, S41, S42, S43, S44, S45, S46, S47, S48, S49, S5, S50, S51, S52, S53, S54, S55, S56, S57, S58, S59, S6, S60, S61, S62, S63, S7, S8, S9: LCSC C9900021274 -> C41430893
Changed lines of the file:
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@@
 			)
 		)
-		(property "LCSC" "C9900021274"
+		(property "LCSC" "C41430893"
 			(at 239.268 97.028 0)
 			(effects
@@
 			)
 		)
-		(property "LCSC" "C9900021274"
+		(property "LCSC" "C41430893"
 			(at 207.518 97.028 0)
 			(effects
@@
 			)
 		)
-		(property "LCSC" "C9900021274"
+		(property "LCSC" "C41430893"
 			(at 158.496 119.126 0)
 			(effects
@@
 			)
 		)
-		(property "LCSC" "C9900021274"
+		(property "LCSC" "C41430893"
 			(at 271.272 74.422 0)
 			(effects
@@
 			)
 		)
-		(property "LCSC" "C9900021274"
+		(property "LCSC" "C41430893"
 			(at 111.252 119.126 0)
 			(effects
@@
 			)
 		)
-		(property "LCSC" "C9900021274"
+		(property "LCSC" "C41430893"
 			(at 271.272 183.642 0)
 			(effects
@@
 			)
 		)
-		(property "LCSC" "C9900021274"
+		(property "LCSC" "C41430893"
 			(at 126.492 97.028 0)
 			(effects
@@
 			)
 		)
-		(property "LCSC" "C9900021274"
+		(property "LCSC" "C41430893"
 			(at 111.252 140.97 0)
 			(effects
@@
 			)
 		)
-		(property "LCSC" "C9900021274"
+		(property "LCSC" "C41430893"
 			(at 224.028 140.97 0)
 			(effects
@@
 			)
 		)
-		(property "LCSC" "C9900021274"
+		(property "LCSC" "C41430893"
 			(at 175.006 162.306 0)
 			(effects
@@
 			)
 		)
-		(property "LCSC" "C9900021274"
+		(property "LCSC" "C41430893"
 			(at 111.252 162.306 0)
 			(effects
@@
 			)
 		)
-		(property "LCSC" "C9900021274"
+		(property "LCSC" "C41430893"
 			(at 271.272 119.126 0)
 			(effects
@@
 			)
 		)
-		(property "LCSC" "C9900021274"
+		(property "LCSC" "C41430893"
 			(at 255.778 162.306 0)
 			(effects
@@
 			)
 		)
-		(property "LCSC" "C9900021274"
+		(property "LCSC" "C41430893"
 			(at 190.246 140.97 0)
 			(effects
@@
 			)
 		)
-		(property "LCSC" "C9900021274"
+		(property "LCSC" "C41430893"
 			(at 94.742 97.028 0)
 			(effects
@@
 			)
 		)
-		(property "LCSC" "C9900021274"
+		(property "LCSC" "C41430893"
 			(at 190.246 162.306 0)
 			(effects
@@
 			)
 		)
-		(property "LCSC" "C9900021274"
+		(property "LCSC" "C41430893"
 			(at 255.778 74.422 0)
 			(effects
@@
 			)
 		)
-		(property "LCSC" "C9900021274"
+		(property "LCSC" "C41430893"
 			(at 175.006 119.126 0)
 			(effects
@@
 			)
 		)
-		(property "LCSC" "C9900021274"
+		(property "LCSC" "C41430893"
 			(at 143.002 140.97 0)
 			(effects
@@
 			)
 		)
-		(property "LCSC" "C9900021274"
+		(property "LCSC" "C41430893"
 			(at 143.002 119.126 0)
 			(effects
@@
 			)
 		)
-		(property "LCSC" "C9900021274"
+		(property "LCSC" "C41430893"
 			(at 224.028 97.028 0)
 			(effects
@@
 			)
 		)
-		(property "LCSC" "C9900021274"
+		(property "LCSC" "C41430893"
 			(at 158.496 74.422 0)
 			(effects
@@
 			)
 		)
-		(property "LCSC" "C9900021274"
+		(property "LCSC" "C41430893"
 			(at 239.268 183.642 0)
 			(effects
@@
 			)
 		)
-		(property "LCSC" "C9900021274"
+		(property "LCSC" "C41430893"
 			(at 287.782 119.126 0)
 			(effects
@@
 			)
 		)
-		(property "LCSC" "C9900021274"
+		(property "LCSC" "C41430893"
 			(at 239.268 162.306 0)
 			(effects
@@
 			)
 		)
-		(property "LCSC" "C9900021274"
+		(property "LCSC" "C41430893"
 			(at 207.518 140.97 0)
 			(effects
@@
 			)
 		)
-		(property "LCSC" "C9900021274"
+		(property "LCSC" "C41430893"
 			(at 126.492 74.422 0)
 			(effects
@@
 			)
 		)
-		(property "LCSC" "C9900021274"
+		(property "LCSC" "C41430893"
 			(at 287.782 74.422 0)
 			(effects
@@
 			)
 		)
-		(property "LCSC" "C9900021274"
+		(property "LCSC" "C41430893"
 			(at 271.272 140.97 0)
 			(effects
@@
 			)
 		)
-		(property "LCSC" "C9900021274"
+		(property "LCSC" "C41430893"
 			(at 303.022 74.422 0)
 			(effects
@@
 			)
 		)
-		(property "LCSC" "C9900021274"
+		(property "LCSC" "C41430893"
 			(at 111.252 97.028 0)
 			(effects
@@
 			)
 		)
-		(property "LCSC" "C9900021274"
+		(property "LCSC" "C41430893"
 			(at 190.246 74.422 0)
 			(effects
@@
 			)
 		)
-		(property "LCSC" "C9900021274"
+		(property "LCSC" "C41430893"
 			(at 126.492 162.306 0)
 			(effects
@@
 			)
 		)
-		(property "LCSC" "C84264"
+		(property "LCSC" "C965805"
 			(at 153.924 225.425 0)
 			(effects
@@
 			)
 		)
-		(property "LCSC" "C9900021274"
+		(property "LCSC" "C41430893"
 			(at 224.028 162.306 0)
 			(effects
@@
 			)
 		)
-		(property "LCSC" "C9900021274"
+		(property "LCSC" "C41430893"
 			(at 190.246 119.126 0)
 			(effects
@@
 			)
 		)
-		(property "LCSC" "C9900021274"
+		(property "LCSC" "C41430893"
 			(at 207.518 119.126 0)
 			(effects
@@
 			)
 		)
-		(property "LCSC" "C9900021274"
+		(property "LCSC" "C41430893"
 			(at 158.496 140.97 0)
 			(effects
@@
 			)
 		)
-		(property "LCSC" "C9900021274"
+		(property "LCSC" "C41430893"
 			(at 207.518 74.422 0)
 			(effects
@@
 			)
 		)
-		(property "LCSC" "C9900021274"
+		(property "LCSC" "C41430893"
 			(at 143.002 162.306 0)
 			(effects
@@
 			)
 		)
-		(property "LCSC" "C9900021274"
+		(property "LCSC" "C41430893"
 			(at 158.496 97.028 0)
 			(effects
@@
 			)
 		)
-		(property "LCSC" "C9900021274"
+		(property "LCSC" "C41430893"
 			(at 287.782 97.028 0)
 			(effects
@@
 			)
 		)
-		(property "LCSC" "C9900021274"
+		(property "LCSC" "C41430893"
 			(at 207.518 162.306 0)
 			(effects
@@
 			)
 		)
-		(property "LCSC" "C9900021274"
+		(property "LCSC" "C41430893"
 			(at 271.272 97.028 0)
 			(effects
@@
 			)
 		)
-		(property "LCSC" "C9900021274"
+		(property "LCSC" "C41430893"
 			(at 175.006 74.422 0)
 			(effects
@@
 			)
 		)
-		(property "LCSC" "C9900021274"
+		(property "LCSC" "C41430893"
 			(at 239.268 74.422 0)
 			(effects
@@
 			)
 		)
-		(property "LCSC" "C9900021274"
+		(property "LCSC" "C41430893"
 			(at 239.268 140.97 0)
 			(effects
@@
 			)
 		)
-		(property "LCSC" "C9900021274"
+		(property "LCSC" "C41430893"
 			(at 239.268 119.126 0)
 			(effects
@@
 			)
 		)
-		(property "LCSC" "C9900021274"
+		(property "LCSC" "C41430893"
 			(at 175.006 97.028 0)
 			(effects
@@
 			)
 		)
-		(property "LCSC" "C9900021274"
+		(property "LCSC" "C41430893"
 			(at 111.252 183.642 0)
 			(effects
@@
 			)
 		)
-		(property "LCSC" "C9900021274"
+		(property "LCSC" "C41430893"
 			(at 255.778 140.97 0)
 			(effects
@@
 			)
 		)
-		(property "LCSC" "C9900021274"
+		(property "LCSC" "C41430893"
 			(at 255.778 97.028 0)
 			(effects
@@
 			)
 		)
-		(property "LCSC" "C9900021274"
+		(property "LCSC" "C41430893"
 			(at 126.492 119.126 0)
 			(effects
@@
 			)
 		)
-		(property "LCSC" "C9900021274"
+		(property "LCSC" "C41430893"
 			(at 224.028 74.422 0)
 			(effects
@@
 			)
 		)
-		(property "LCSC" "C9900021274"
+		(property "LCSC" "C41430893"
 			(at 143.002 74.422 0)
 			(effects
@@
 			)
 		)
-		(property "LCSC" "C9900021274"
+		(property "LCSC" "C41430893"
 			(at 255.778 119.126 0)
 			(effects
@@
 			)
 		)
-		(property "LCSC" "C9900021274"
+		(property "LCSC" "C41430893"
 			(at 126.492 140.97 0)
 			(effects
@@
 			)
 		)
-		(property "LCSC" "C9900021274"
+		(property "LCSC" "C41430893"
 			(at 158.496 162.306 0)
 			(effects
@@
 			)
 		)
-		(property "LCSC" "C9900021274"
+		(property "LCSC" "C41430893"
 			(at 255.778 183.642 0)
 			(effects
@@
 			)
 		)
-		(property "LCSC" "C9900021274"
+		(property "LCSC" "C41430893"
 			(at 175.006 140.97 0)
 			(effects
@@
 			)
 		)
-		(property "LCSC" "C9900021274"
+		(property "LCSC" "C41430893"
 			(at 190.246 97.028 0)
 			(effects
@@
 			)
 		)
-		(property "LCSC" "C9900021274"
+		(property "LCSC" "C41430893"
 			(at 94.742 74.422 0)
 			(effects
@@
 			)
 		)
-		(property "LCSC" "C9900021274"
+		(property "LCSC" "C41430893"
 			(at 224.028 119.126 0)
 			(effects
@@
 			)
 		)
-		(property "LCSC" "C9900021274"
+		(property "LCSC" "C41430893"
 			(at 143.002 97.028 0)
 			(effects
