File: kicad/GlyphMatrix-keymatrix.kicad_sch (KiCad schematic)
At the start: 169 parts

Commit message: more updates (#12)
* working on kibot

* added position file

* fixed footprint for PhaseShift and DeltaForm

* fixed footprint side for GlyphMatrix

* KiBot: changed BOM type

* added fonts

* KiBot

* refreshed submodule

* updated footprint for GlyphMatrix

* updated footprint for PhaseShift

* updated footprint for DeltaForm

* updated build guide
Parts:
- S64, S65, S66, S67, S68, S69, S70, S71, S72, S73, S74: LCSC C9900021274 -> C41430893
Changed lines of the file:
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@@
 			)
 		)
-		(property "LCSC" "C9900021274"
+		(property "LCSC" "C41430893"
 			(at 303.022 140.97 0)
 			(effects
@@
 			)
 		)
-		(property "LCSC" "C9900021274"
+		(property "LCSC" "C41430893"
 			(at 303.022 183.642 0)
 			(effects
@@
 			)
 		)
-		(property "LCSC" "C9900021274"
+		(property "LCSC" "C41430893"
 			(at 94.742 140.97 0)
 			(effects
@@
 			)
 		)
-		(property "LCSC" "C9900021274"
+		(property "LCSC" "C41430893"
 			(at 119.634 190.5 0)
 			(effects
@@
 			)
 		)
-		(property "LCSC" "C9900021274"
+		(property "LCSC" "C41430893"
 			(at 303.022 162.306 0)
 			(effects
@@
 			)
 		)
-		(property "LCSC" "C9900021274"
+		(property "LCSC" "C41430893"
 			(at 94.742 162.306 0)
 			(effects
@@
 			)
 		)
-		(property "LCSC" "C9900021274"
+		(property "LCSC" "C41430893"
 			(at 94.742 183.642 0)
 			(effects
@@
 			)
 		)
-		(property "LCSC" "C9900021274"
+		(property "LCSC" "C41430893"
 			(at 303.022 97.028 0)
 			(effects
@@
 			)
 		)
-		(property "LCSC" "C9900021274"
+		(property "LCSC" "C41430893"
 			(at 303.022 119.126 0)
 			(effects
@@
 			)
 		)
-		(property "LCSC" "C9900021274"
+		(property "LCSC" "C41430893"
 			(at 94.742 119.126 0)
 			(effects
@@
 			)
 		)
-		(property "LCSC" "C9900021274"
+		(property "LCSC" "C41430893"
 			(at 175.006 183.642 0)
 			(effects

Commit message: reorg schematic for GlyphMatrix
Parts:
- removed D1, D10, D11, D12, D13, D14, D15, D16, D17, D18, D19, D2, D20, D21, D22, D23, D24, D25, D26, D27, D28, D29, D3, D30, D31, D32, D33, D34, D35, D36, D37, D38, D39, D4, D40, D41, D42, D43, D44, D45, D46, D47, D48, D49, D5, D50, D51, D52, D53, D54, D55, D56, D57, D58, D59, D6, D60, D61, D62, D63, D64, D65, D66, D67, D68, D69, D7, D70, D71, D72, D73, D74, D8, D9: 1N4148W, TB2086_SMD:D3_SMD, symbol Device:D
- removed H1, H2, H3, H4, H5, H6, H7, H8: MountingHole_Pad, TB2086_MISC:MountingHole_2.2mm_M2_Pad, symbol TB2086_MISC:MountingHole_Pad
- removed LED2: GREEN, LED_SMD:LED_0603_1608Metric_Pad1.05x0.95mm_HandSolder, symbol Device:LED
- removed POGO1, POGO2: Conn_01x05, TB2086_MISC:Pogopin_1x05_P2.54mm_Curved, symbol Connector_Generic:Conn_01x05
- removed POGO3, POGO4, POGO5, POGO6: Conn_01x07, TB2086_MISC:Pogopin_1x07_P2.54mm_Curved, symbol Connector_Generic:Conn_01x07
- removed R9: 330, Resistor_SMD:R_0603_1608Metric, symbol Device:R_Small
- removed S1, S10, S11, S12, S13, S14, S15, S16, S17, S18, S19, S2, S20, S21, S22, S23, S24, S25, S26, S27, S28, S29, S3, S30, S31, S32, S33, S34, S35, S36, S37, S38, S39, S4, S40, S41, S42, S43, S44, S45, S46, S47, S48, S49, S5, S50, S51, S52, S53, S54, S55, S56, S57, S58, S59, S6, S60, S61, S62, S63, S7, S8, S9: SW_MX_HS, TB2086_KEYSWITCH:SW_MX_HS_1u, symbol TB2086_KEYSWITCH:SW_MX_HS
- removed S64: SW_MX_HS, TB2086_KEYSWITCH:SW_MX_HS_1.25u, symbol TB2086_KEYSWITCH:SW_MX_HS
- removed S65, S66: SW_MX_HS, TB2086_KEYSWITCH:SW_MX_HS_1.5u, symbol TB2086_KEYSWITCH:SW_MX_HS
- removed S67, S68, S69: SW_MX_HS, TB2086_KEYSWITCH:SW_MX_HS_1.75u, symbol TB2086_KEYSWITCH:SW_MX_HS
- removed S70: SW_MX_HS, TB2086_KEYSWITCH:SW_MX_HS_2u, symbol TB2086_KEYSWITCH:SW_MX_HS
- removed S71, S72: SW_MX_HS, TB2086_KEYSWITCH:SW_MX_HS_2.25u, symbol TB2086_KEYSWITCH:SW_MX_HS
- removed S73: SW_MX_HS, TB2086_KEYSWITCH:SW_MX_HS_2.75u, symbol TB2086_KEYSWITCH:SW_MX_HS
- removed S74: SW_MX_HS, TB2086_KEYSWITCH:SW_MX_HS_6.25u, symbol TB2086_KEYSWITCH:SW_MX_HS
- removed STB1, STB2, STB3, STB4: Stabilizer_Cherry_MX_2.00u, Stabilizer_Cherry_MX_2.00u, symbol PCM_marbastlib-mx:MX_stab
- removed STB5: Stabilizer_Cherry_MX_6.25u, Stabilizer_Cherry_MX_6.25u, symbol PCM_marbastlib-mx:MX_stab
