File: kicad/PhaseShift.kicad_pcb (KiCad board)
At the start: 2 copper layers, 66.4 x 128.6 mm, 56 parts

Commit message: small tweaks
Parts:
- moved LED1 19.1 mm to (204.5, 101.9)
- moved R1 19.1 mm to (204.5, 101.9)
Routing:
- net COL1: track 181.3 -> 186.9 mm
- net COL0: track 177.9 -> 172.6 mm
- net COL2: track 181.8 -> 176.6 mm
- net SCR: track 77.6 -> 75.7 mm, vias 0 -> 1
- net Net-(L4-DOUT): track 30.1 -> 30.9 mm
- net +5V: track 318.1 -> 318.6 mm
Other:
- board text added: "OmniCode:9001 - 202507.10"
- board text removed: "OmniCode:9001 - 202507.09"

Commit message: PhaseShift - 3mm screws
Parts:
- H1, H2, H3, H4, H5: value MountingHole_2.2mm_M2_Pad -> MountingHole_3.2mm_Pad; footprint TB2086_MISC:MountingHole_2.2mm_M2_Pad -> TB2086_MISC:MountingHole_3.2mm_Pad
- moved H1 0.71 mm to (175.8, 80.2)
- moved H2 0.71 mm to (233.2, 80.2)
- moved H3 0.71 mm to (233.2, 199.8)
- moved H4 0.71 mm to (175.8, 199.8)
Other:
- board text added: "OmniCode:9001 - 202507.12"
- board text removed: "OmniCode:9001 - 202507.10"

Commit message: fixed footprint for PhaseShift and DeltaForm
Parts:
- S1, S10, S11, S12, S13, S2, S3, S4, S5, S6, S7, S8, S9: moved to B.Cu
- turned S1 to 0 degrees
- turned S10 to 0 degrees
- turned S11 to 0 degrees
- turned S12 to 0 degrees
- turned S13 to 0 degrees
- turned S2 to 0 degrees
- turned S3 to 0 degrees
- turned S4 to 0 degrees
- turned S5 to 0 degrees
- turned S6 to 0 degrees
- turned S7 to 0 degrees
- turned S8 to 0 degrees
- turned S9 to 0 degrees
