File: kicad/GlyphMatrix.kicad_pcb (KiCad board)
At the start: 2 copper layers, 294.9 x 128.6 mm, 281 parts, among them J1 Conn_01x04, SW1 SW_Push, SW2 SW_Push, U1 W25Q128JVS, U2 USBLC6-2SC6, U3 XC6206PxxxMR-Regulator_Linear, Y1 12MHz

Commit message: adjusted positions
- pogo pins
Parts:
- moved POGO1 0.45 mm to (64.5, 95.5)
- moved POGO3 0.45 mm to (64.5, 142.4)
- moved POGO5 0.45 mm to (64.5, 182.0)
- moved POGO2 0.45 mm to (352.1, 95.5)
- moved POGO4 0.45 mm to (352.1, 142.4)
- moved POGO6 0.45 mm to (352.1, 182.0)
Routing:
- net COL1: track 579.0 -> 588.3 mm, vias 8 -> 7
- net Net-(L27-DIN): track 36.0 -> 27.1 mm
- net COL2: track 636.9 -> 638.5 mm
- net COL0: track 627.5 -> 628.8 mm
- net ROW11: track 175.3 -> 174.1 mm
- net ROW13: track 495.5 -> 496.6 mm
- net ROW02: track 298.9 -> 300.0 mm
- net RGB_FOM_RIGHT: track 94.4 -> 95.4 mm
- net +5V: track 1828.5 -> 1829.2 mm

Commit message: small tweak
- pogo pin
Parts:
- moved POGO1 0.12 mm to (64.7, 95.5)
- moved POGO2 0.12 mm to (352.0, 95.5)
- moved POGO3 0.12 mm to (64.7, 142.4)
- moved POGO4 0.12 mm to (352.0, 142.4)
- moved POGO5 0.12 mm to (64.7, 182.0)
- moved POGO6 0.12 mm to (352.0, 182.0)
Changed lines of the file:
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@@
 	(footprint "TB2086_MISC:Pogopin_1x07_P2.54mm_Curved"
 		(layer "B.Cu")
-		(at 64.55 182 -90)
+		(at 64.675 182 -90)
 		(property "Reference" "POGO5"
 			(at 0 1.77 90)
@@
 	(footprint "TB2086_MISC:Pogopin_1x07_P2.54mm_Curved"
 		(layer "B.Cu")
-		(at 352.15 182 90)
+		(at 352.025 182 90)
 		(property "Reference" "POGO6"
 			(at 0 1.77 270)
@@
 	(footprint "TB2086_MISC:Pogopin_1x05_P2.54mm_Curved"
 		(layer "B.Cu")
-		(at 352.15 95.5125 90)
+		(at 352.025 95.5125 90)
 		(property "Reference" "POGO2"
 			(at 0 1.77 270)
@@
 	(footprint "TB2086_MISC:Pogopin_1x07_P2.54mm_Curved"
 		(layer "B.Cu")
-		(at 352.15 142.3875 90)
+		(at 352.025 142.3875 90)
 		(property "Reference" "POGO4"
 			(at 0 1.77 270)
@@
 	(footprint "TB2086_MISC:Pogopin_1x05_P2.54mm_Curved"
 		(layer "B.Cu")
-		(at 64.55 95.5125 -90)
+		(at 64.675 95.5125 -90)
 		(property "Reference" "POGO1"
 			(at 0 1.77 90)
@@
 	(footprint "TB2086_MISC:Pogopin_1x07_P2.54mm_Curved"
 		(layer "B.Cu")
-		(at 64.55 142.3875 -90)
+		(at 64.675 142.3875 -90)
 		(property "Reference" "POGO3"
 			(at 0 1.77 90)
@@
 	)
 	(segment
-		(start 352.5625 90.4325)
-		(end 353.91 91.78)
+		(start 353.68 91.55)
+		(end 353.68 110.6325)
 		(width 0.2)
 		(layer "B.Cu")
@@
 	)
 	(segment
-		(start 353.91 91.78)
-		(end 353.91 110.4025)
+		(start 351.7 89.28)
+		(end 351.7 90.4325)
 		(width 0.2)
 		(layer "B.Cu")
@@
 	)
 	(segment
-		(start 351.7 89.28)
-		(end 351.7 90.4325)
+		(start 352.5625 90.4325)
+		(end 353.68 91.55)
 		(width 0.2)
 		(layer "B.Cu")
@@
 	)
 	(segment
-		(start 353.91 110.4025)
+		(start 353.68 110.6325)
 		(end 351.225 113.0875)
 		(width 0.2)
@@
 	)
 	(segment
-		(start 354.29 187.03)
+		(start 351.225 121.405)
+		(end 353.84 124.02)
+		(width 0.2)
+		(layer "B.Cu")
+		(net 138)
+	)
+	(segment
+		(start 352.12 189.62)
 		(end 351.7 189.62)
 		(width 0.2)
@@
 	)
 	(segment
-		(start 351.225 121.405)
-		(end 354.29 124.47)
+		(start 353.84 187.9)
+		(end 352.12 189.62)
 		(width 0.2)
 		(layer "B.Cu")
@@
 	)
 	(segment
-		(start 351.225 114.5375)
-		(end 351.225 121.405)
+		(start 338.7309 182.5017)
+		(end 339.63 182.5017)
 		(width 0.2)
 		(layer "B.Cu")
@@
 	)
 	(segment
-		(start 354.29 124.47)
-		(end 354.29 187.03)
+		(start 353.84 124.02)
+		(end 353.84 187.9)
 		(width 0.2)
 		(layer "B.Cu")
@@
 	)
 	(segment
-		(start 338.7309 182.5017)
-		(end 339.63 182.5017)
+		(start 351.225 114.5375)
+		(end 351.225 121.405)
 		(width 0.2)
 		(layer "B.Cu")
