File: kicad/GlyphMatrix.kicad_pcb (KiCad board)
At the start: 2 copper layers, 294.9 x 128.6 mm, 281 parts, among them J1 Conn_01x04, SW1 SW_Push, SW2 SW_Push, U1 W25Q128JVS, U2 USBLC6-2SC6, U3 XC6206PxxxMR-Regulator_Linear, Y1 12MHz

Commit message: adjust pogo pin positions (#21)
* adjusted positions

* small tweak

* updated ergogen

* 202508.04
Parts:
- moved POGO1 0.33 mm to (64.7, 95.5)
- moved POGO3 0.33 mm to (64.7, 142.4)
- moved POGO5 0.33 mm to (64.7, 182.0)
- moved POGO2 0.32 mm to (352.0, 95.5)
- moved POGO4 0.32 mm to (352.0, 142.4)
- moved POGO6 0.32 mm to (352.0, 182.0)
Routing:
- net COL1: track 579.0 -> 588.3 mm, vias 8 -> 7
- net Net-(L27-DIN): track 36.0 -> 27.1 mm
- net COL2: track 636.9 -> 638.5 mm
- net COL0: track 627.5 -> 628.8 mm
- net ROW11: track 175.3 -> 174.1 mm
- net ROW13: track 495.5 -> 496.6 mm
- net ROW02: track 298.9 -> 300.0 mm
- net RGB_FOM_RIGHT: track 94.4 -> 95.2 mm
- net +5V: track 1828.5 -> 1829.2 mm
Other:
- board text added: "OmniCode:9001 - 202508.04"
- board text removed: "OmniCode:9001 - 202507.22"

Commit message: tweaked zone (#22)
* small tweak

* removed isolated copper islands
Routing:
- net +5V: track 1829.2 -> 2036.8 mm, vias 10 -> 13
- net COL0: track 628.8 -> 591.8 mm
- net ROW03: track 212.9 -> 189.9 mm, vias 6 -> 7
- net COL6: track 575.6 -> 593.1 mm
- net Net-(L31-DIN): track 21.6 -> 35.4 mm
- net Net-(L22-DIN): track 34.5 -> 45.8 mm
- net Net-(L19-DOUT): track 27.1 -> 38.3 mm
- net ROW17: track 492.0 -> 501.8 mm
- net Net-(L11-DIN): track 29.2 -> 37.4 mm
- net Net-(L32-DOUT): track 30.3 -> 22.8 mm
- net COL5: track 665.9 -> 673.2 mm
- net ROW12: track 498.1 -> 505.4 mm
- net Net-(L66-DOUT): track 21.6 -> 28.7 mm
- net ROW06: track 283.8 -> 277.5 mm
- net ROW16: track 492.4 -> 498.6 mm
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Other:
- board text added: "Bloomberg"
- board text added: "Engineering"
