File: kicad/GlyphMatrix.kicad_pcb (KiCad board)
At the start: 2 copper layers, 294.9 x 128.6 mm, 281 parts, among them J1 Conn_01x04, SW1 SW_Push, SW2 SW_Push, U1 W25Q128JVS, U2 USBLC6-2SC6, U3 XC6206PxxxMR-Regulator_Linear, Y1 12MHz

Commit message: 202508.10
Other:
- board text added: "OmniCode:9001 - 202508.10"
- board text removed: "OmniCode:9001 - 202508.04"

Commit message: side bars
Other:
- board text removed: "Bloomberg"
- board text removed: "Engineering"
