File: kicad/DeltaForm.kicad_pcb (KiCad board)
At the start: 2 copper layers, 85.4 x 128.6 mm, 82 parts

Commit message: adjust pogo pin positions (#21)
* adjusted positions

* small tweak

* updated ergogen

* 202508.04
Parts:
- moved POGO1 0.33 mm to (167.0, 95.5)
- moved POGO2 0.33 mm to (244.8, 95.5)
- moved POGO3 0.33 mm to (167.0, 142.4)
- moved POGO4 0.33 mm to (244.8, 142.4)
- moved POGO5 0.33 mm to (167.0, 182.0)
- moved POGO6 0.33 mm to (244.8, 182.0)
Routing:
- net COL3: track 217.4 -> 214.5 mm
- net ROW12: track 227.8 -> 229.2 mm
- net ROW13: track 180.9 -> 179.6 mm
- net ROW17: track 99.6 -> 100.4 mm
- net COL4: track 182.6 -> 183.2 mm
Other:
- board text added: "OmniCode:9001 - 202508.04"
- board text removed: "OmniCode:9001 - 202507.22"
