File: kicad/GlyphMatrix.kicad_sch (KiCad schematic)
At the start: 167 parts

Commit message: fixed mounting hole for GlyphMatrix (#27)
Parts:
- H1, H2, H3, H4, H5, H6, H7, H8: footprint TB2086_MISC:MountingHole_2.2mm_M2_Pad -> TB2086_MISC:MountingHole_3.2mm_Pad
Changed lines of the file:
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@@
 			)
 		)
-		(property "Footprint" "TB2086_MISC:MountingHole_2.2mm_M2_Pad"
+		(property "Footprint" "TB2086_MISC:MountingHole_3.2mm_Pad"
 			(at 82.55 221.742 0)
 			(effects
@@
 			)
 		)
-		(property "Footprint" "TB2086_MISC:MountingHole_2.2mm_M2_Pad"
+		(property "Footprint" "TB2086_MISC:MountingHole_3.2mm_Pad"
 			(at 82.55 232.918 0)
 			(effects
@@
 			)
 		)
-		(property "Footprint" "TB2086_MISC:MountingHole_2.2mm_M2_Pad"
+		(property "Footprint" "TB2086_MISC:MountingHole_3.2mm_Pad"
 			(at 82.55 204.216 0)
 			(effects
@@
 			)
 		)
-		(property "Footprint" "TB2086_MISC:MountingHole_2.2mm_M2_Pad"
+		(property "Footprint" "TB2086_MISC:MountingHole_3.2mm_Pad"
 			(at 82.55 210.312 0)
 			(effects
@@
 			)
 		)
-		(property "Footprint" "TB2086_MISC:MountingHole_2.2mm_M2_Pad"
+		(property "Footprint" "TB2086_MISC:MountingHole_3.2mm_Pad"
 			(at 82.55 191.516 0)
 			(effects
@@
 			)
 		)
-		(property "Footprint" "TB2086_MISC:MountingHole_2.2mm_M2_Pad"
+		(property "Footprint" "TB2086_MISC:MountingHole_3.2mm_Pad"
 			(at 82.55 215.646 0)
 			(effects
@@
 			)
 		)
-		(property "Footprint" "TB2086_MISC:MountingHole_2.2mm_M2_Pad"
+		(property "Footprint" "TB2086_MISC:MountingHole_3.2mm_Pad"
 			(at 82.55 197.612 0)
 			(effects
@@
 			)
 		)
-		(property "Footprint" "TB2086_MISC:MountingHole_2.2mm_M2_Pad"
+		(property "Footprint" "TB2086_MISC:MountingHole_3.2mm_Pad"
 			(at 82.55 226.822 0)
 			(effects
